File: PCB/BinMonitored.brd (EAGLE design)
At the start: 25.4 x 25.4 mm, 30 parts, among them U1 VL53L1XSMD, U2 24LC256, U3 MMA8452Q, U4 3.3V, U5 BME680

Commit message: Tidied up Schematic and added measurements to the PCB.
Parts:
- added FRAME1: FRAME-LEDGER, SparkFun-Aesthetics:CREATIVE_COMMONS
- R8: value (none) -> 39k
- R9: value (none) -> 10k

Commit message: Tidyuip for values and text.
Parts:
- C5, C6: value 0.1uF -> 1.0uF
- U2: value 24LC256 -> 24LC512
Changed lines of the file:
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@@
 <dimension x1="12.7" y1="3.175" x2="0" y2="3.8" x3="6.35" y3="-5.6" textsize="1.778" layer="47" dtype="horizontal"/>
 <dimension x1="12.7" y1="3.175" x2="12.3" y2="0" x3="-1.7" y3="1.5875" textsize="1.778" layer="47" dtype="vertical"/>
+<dimension x1="10.16" y1="19.05" x2="0" y2="18.2" x3="5.08" y3="35.5" textsize="1.778" layer="47" dtype="horizontal"/>
+<dimension x1="10.16" y1="19.05" x2="9" y2="0" x3="-8.1" y3="9.525" textsize="1.778" layer="47" dtype="vertical"/>
+<dimension x1="10.16" y1="19.05" x2="10.2" y2="21.5" x3="-8.1" y3="20.275" textsize="1.778" layer="47" dtype="vertical"/>
+<dimension x1="10.16" y1="19.05" x2="11.7" y2="21" x3="10.93" y3="35.5" textsize="1.778" layer="47" dtype="horizontal"/>
 </plain>
 <attributes>
@@
 <attribute name="VALUE" x="23.495" y="22.987" size="0.6096" layer="27" font="vector" ratio="20" rot="R180" align="top-center"/>
 </element>
-<element name="C5" library="SparkFun-Capacitors" package="0603" value="0.1uF" x="17.145" y="9.525" smashed="yes" rot="R270">
+<element name="C5" library="SparkFun-Capacitors" package="0603" value="1.0uF" x="17.145" y="9.525" smashed="yes" rot="R270">
 <attribute name="PROD_ID" value="CAP-08604" x="17.145" y="9.525" size="1.778" layer="27" rot="R270" display="off"/>
 <attribute name="NAME" x="17.145" y="11.3395" size="0.6096" layer="25" font="vector" ratio="20" align="bottom-center"/>
 <attribute name="VALUE" x="17.145" y="9.3345" size="0.6096" layer="27" font="vector" ratio="20" rot="R180" align="top-center"/>
 </element>
-<element name="C6" library="SparkFun-Capacitors" package="0603" value="0.1uF" x="21.59" y="1.905" smashed="yes">
+<element name="C6" library="SparkFun-Capacitors" package="0603" value="1.0uF" x="21.59" y="1.905" smashed="yes">
 <attribute name="PROD_ID" value="CAP-08604" x="21.59" y="1.905" size="1.778" layer="27" display="off"/>
 <attribute name="NAME" x="19.7505" y="1.8725" size="0.6096" layer="25" font="vector" ratio="20" rot="R90" align="bottom-center"/>
 <attribute name="VALUE" x="21.9505" y="2.295" size="0.6096" layer="27" font="vector" ratio="20" rot="R270" align="top-center"/>
 </element>
-<element name="U2" library="SparkFun-IC-Memory" package="SO08" value="24LC256" x="4.445" y="3.81" smashed="yes">
+<element name="U2" library="SparkFun-IC-Memory" package="SO08" value="24LC512" x="4.445" y="3.81" smashed="yes">
 <attribute name="PROD_ID" value="IC-09714" x="4.445" y="3.81" size="1.778" layer="27" ratio="16" display="off"/>
 <attribute name="NAME" x="4.1275" y="5.3975" size="0.6096" layer="25" font="vector" ratio="20" rot="R180" align="bottom-center"/>
