File: PCB/BinMonitored.sch (EAGLE design)
At the start: 30 parts, among them U1 VL53L1XSMD, U2 24LC256, U3 MMA8452Q, U4 3.3V, U5 BME680

Commit message: Tidied up Schematic and added measurements to the PCB.
Parts:
- added FRAME1: FRAME-LEDGER, SparkFun-Aesthetics:FRAME-LEDGER
- R8: value (none) -> 39k
- R9: value (none) -> 10k
Other:
- note added: "Accelerometer (Lid Lift) Sensor"
- note added: "Approx. 1/5 of the battery voltage (4.2 ->0.84v) to the ESP's ADC which has the rante 0-1V over 10 bits (max 1023)."
- note added: "Battery Monitor"
- note added: "Bin Monitored"
- note added: "Distance Sensor"
- note added: "EEPROM Memory"
- note added: "ESP Programming Connections"
- note added: "ESP-12 MicroController"
- note added: "Environmental Sensor"
- note added: "I2C Pullups"
- note added: "Monitor your wheelie bin. * Has it fallen over * Has the delivery person left a parcel in it * Is your neighbour putting their rubbish in it? * Is it hot/cold or very wet? * How full is it?"
- note added: "Power Connector"
- note added: "Stephen Harrison"
- note added: "Use a LiPol (3.6-4.2V Battery)"
- note added: "V1.0"
- note added: "Voltage Regulator"
- moved on the sheet: C3, C4, C5, C6, D0, D1, D2, GND, J1, R, R4, R5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

Commit message: Tidyuip for values and text.
Parts:
- C5, C6: value 0.1uF -> 1.0uF
- U2: value 24LC256 -> 24LC512
Other:
- note added: "Addr: 0x1D"
- note added: "Addr: 0x50"
- note added: "Conformal Coating: RS: 535-525 https://uk.rs-online.com/web/p/conformal-coatings/0535525/"
Changed lines of the file:
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@@
 <part name="SUPPLY18" library="SparkFun-PowerSymbols" deviceset="V_BATT" device=""/>
 <part name="GND17" library="SparkFun-PowerSymbols" deviceset="GND" device=""/>
-<part name="C5" library="SparkFun-Capacitors" deviceset="0.1UF" device="-0603-25V-5%" value="0.1uF"/>
-<part name="C6" library="SparkFun-Capacitors" deviceset="0.1UF" device="-0603-25V-5%" value="0.1uF"/>
+<part name="C5" library="SparkFun-Capacitors" deviceset="0.1UF" device="-0603-25V-5%" value="1.0uF"/>
+<part name="C6" library="SparkFun-Capacitors" deviceset="0.1UF" device="-0603-25V-5%" value="1.0uF"/>
 <part name="SUPPLY19" library="SparkFun-PowerSymbols" deviceset="V_BATT" device=""/>
 <part name="GND18" library="SparkFun-PowerSymbols" deviceset="GND" device=""/>
 <part name="SUPPLY20" library="SparkFun-PowerSymbols" deviceset="3.3V" device=""/>
 <part name="GND19" library="SparkFun-PowerSymbols" deviceset="GND" device=""/>
-<part name="U2" library="SparkFun-IC-Memory" deviceset="EEPROM-I2C" device="SMD" value="24LC256"/>
+<part name="U2" library="SparkFun-IC-Memory" deviceset="EEPROM-I2C" device="SMD" value="24LC512"/>
 <part name="SUPPLY21" library="SparkFun-PowerSymbols" deviceset="3.3V" device=""/>
 <part name="GND7" library="SparkFun-PowerSymbols" deviceset="GND" device=""/>
@@
 * How full is it?
 </text>
+<text x="198.12" y="154.94" size="1.778" layer="97">Conformal Coating:
+RS: 535-525
+https://uk.rs-online.com/web/p/conformal-coatings/0535525/</text>
+<text x="-76.2" y="-12.7" size="1.27" layer="97">Addr: 0x50</text>
+<text x="0" y="-50.8" size="1.27" layer="97">Addr: 0x1D</text>
 </plain>
 <instances>
